File: pcb/6502_v1.kicad_sch (KiCad schematic)
At the start: 95 parts, among them J1 Jack-DC, J10 V_SLCT, J11 ACPort2, J12 WE_Cont, J2 Screw_Terminal_01x02, J3 VBus-80, J4 NMI_Contr, J5 JTAG, J6 KeyboardCon, J7 PORTA, J8 PORTB, J9 ACPort1, Q1 NMOS, Q2 NMOS, Q3 NMOS, Q4 NMOS, Q5 NMOS, Q6 NMOS, Q7 NMOS, Q8 NMOS, SW1 SW_Push, U1 74HC14, U10 L7805, U11 LD1117V33, U12 74HC595, U14 6522, U15 6502, U2 28C256, U3 CY62256-70PC, U5 6522, U6 W65C51NxP, U7 W65C51NxP, U8 EPM7128SLC84-15, U9 74AHC595, Y1 1.8432mHz, Y2 50mHz, Y3 Crystal

Commit message: V4 Pcb Upload.
Parts:
- removed C98, C99: 0.1uF, Capacitor_THT:C_Disc_D3.4mm_W2.1mm_P2.50mm, symbol Device:C
- removed D6: SB140, Diode_THT:D_DO-41_SOD81_P10.16mm_Horizontal, symbol Diode:SB140
- removed D8: 1N4001, Diode_THT:D_DO-41_SOD81_P10.16mm_Horizontal, symbol Diode:1N4001
- removed J1: Jack-DC, Connector_BarrelJack:BarrelJack_GCT_DCJ200-10-A_Horizontal, symbol Connector:Jack-DC
- removed J10: V_SLCT, Connector_PinHeader_2.54mm:PinHeader_1x03_P2.54mm_Vertical, symbol Connector_Generic:Conn_01x03
- removed J11: ACPort2, Connector_PinSocket_2.54mm:PinSocket_1x04_P2.54mm_Horizontal, symbol Connector_Generic:Conn_01x04
- removed J12: WE_Cont, Connector_PinHeader_2.54mm:PinHeader_1x03_P2.54mm_Vertical, symbol Connector_Generic:Conn_01x03
- removed J2: Screw_Terminal_01x02, TerminalBlock:TerminalBlock_bornier-2_P5.08mm, symbol Connector:Screw_Terminal_01x02
- removed J3: VBus-80, Connector_PinSocket_2.54mm:PinSocket_2x40_P2.54mm_Horizontal, symbol Connector_Generic:Conn_02x40_Odd_Even
- removed J4: NMI_Contr, Connector_PinHeader_2.54mm:PinHeader_1x03_P2.54mm_Vertical, symbol Connector_Generic:Conn_01x03
- removed J5: JTAG, Connector_PinHeader_2.54mm:PinHeader_2x05_P2.54mm_Vertical, symbol Connector_Generic:Conn_02x05_Odd_Even
- removed J6: KeyboardCon, Connector_PinSocket_2.54mm:PinSocket_1x05_P2.54mm_Horizontal, symbol Connector_Generic:Conn_01x05
- removed J8: PORTB, Connector_PinSocket_2.54mm:PinSocket_2x09_P2.54mm_Horizontal, symbol Connector_Generic:Conn_02x09_Odd_Even
- removed J9: ACPort1, Connector_PinSocket_2.54mm:PinSocket_1x04_P2.54mm_Horizontal, symbol Connector_Generic:Conn_01x04
- removed Q1, Q2, Q3, Q4, Q5, Q6, Q7, Q8: NMOS, Package_TO_SOT_THT:TO-92_Inline, symbol Simulation_SPICE:NMOS
- removed R10, R11, R12, R16, R17, R18, R19, R20, R21, R7, R8, R9: 10k, Resistor_THT:R_Axial_DIN0207_L6.3mm_D2.5mm_P10.16mm_Horizontal, symbol Device:R
- removed R14: 1K, Resistor_THT:R_Axial_DIN0207_L6.3mm_D2.5mm_P10.16mm_Horizontal, symbol Device:R
- removed R15: 10K, Resistor_THT:R_Axial_DIN0207_L6.3mm_D2.5mm_P10.16mm_Horizontal, symbol Device:R
- removed R25: ?, Resistor_THT:R_Axial_DIN0207_L6.3mm_D2.5mm_P10.16mm_Horizontal, symbol Device:R
- removed R28: R, Resistor_THT:R_Axial_DIN0207_L6.3mm_D2.5mm_P10.16mm_Horizontal, symbol Device:R
- removed U1: 74HC14, Package_DIP:DIP-14_W7.62mm, symbol 74xx:74HC14
- removed U10: L7805, Package_TO_SOT_THT:TO-220-3_Vertical, symbol Regulator_Linear:L7805
- removed U11: LD1117V33, Package_TO_SOT_THT:TO-220-3_Vertical, symbol Regulator_Linear:L7805
- removed U12: 74HC595, Package_DIP:DIP-16_W7.62mm_Socket, symbol 74xx:74HC595
- removed U14: 6522, Package_DIP:DIP-40_W15.24mm_Socket, symbol 65xx-library:6522
- removed U9: 74AHC595, Package_DIP:DIP-16_W7.62mm_Socket, symbol 74xx:74AHC595
- removed Y2: 50mHz, crystal:OSC_ECS-2100AX-200, symbol ECS-2100A-8.0MHZ:ECS-2100A-8.0MHZ
- added C19, C20, C21, C22, C23, C27, C28, C29, C9: 0.01uF, Capacitor_THT:C_Disc_D3.4mm_W2.1mm_P2.50mm, symbol Device:C
- added C30, C31: C, Capacitor_THT:C_Disc_D3.4mm_W2.1mm_P2.50mm, symbol Device:C
- added C32: MainC, Capacitor_THT:CP_Radial_D5.0mm_P2.00mm, symbol Device:C_Polarized
- added C33, C34: C, Capacitor_THT:CP_Radial_D5.0mm_P2.00mm, symbol Device:C_Polarized
- added D11: 1N4001, Diode_THT:D_DO-41_SOD81_P10.16mm_Horizontal, symbol Diode:1N4001
- added D6: D, Diode_THT:D_DO-41_SOD81_P10.16mm_Horizontal, symbol Device:D
- added D8, D9: SB140, Diode_THT:D_DO-41_SOD81_P10.16mm_Horizontal, symbol Diode:SB140
- added F1: Fuse, Fuse:Fuse_2920_7451Metric, symbol Device:Fuse
- added J1: VGA_Out, Connector_Dsub:DSUB-15-HD_Female_Horizontal_P2.29x1.98mm_EdgePinOffset3.03mm_Housed_MountingHolesOffset4.94mm, symbol Connector:DE15_Plug_HighDensity
- added J10: PS2-MINIDIN6-FEMALE, kicad_sym:MINI-DIN-6-FULL-SHIELD, symbol PS2_MINIDIN6_FEMALE:PS2-MINIDIN6-FEMALE
- added J11: JTAG, Connector_PinHeader_2.54mm:PinHeader_2x05_P2.54mm_Vertical, symbol Connector_Generic:Conn_02x05_Odd_Even
- added J12: Debug_CS, Connector_PinHeader_2.54mm:PinHeader_1x04_P2.54mm_Vertical, symbol Connector:Conn_01x04_Socket
- added J13: Debug_ADR1, Connector_PinHeader_2.54mm:PinHeader_1x04_P2.54mm_Vertical, symbol Connector:Conn_01x04_Socket
- added J14: VGA_Conf, Jumper:SolderJumper-3_P1.3mm_Open_RoundedPad1.0x1.5mm_NumberLabels, symbol Connector:Conn_01x02_Pin
- added J15, J17, J18, J19, J20, J21, J22, J23, J24: PW_JMP, Connector_PinSocket_2.54mm:PinSocket_1x01_P2.54mm_Vertical, symbol Connector:Conn_01x01_Pin
- added J16, J6: EN, Jumper:SolderJumper-3_P1.3mm_Open_RoundedPad1.0x1.5mm_NumberLabels, symbol Connector:Conn_01x02_Pin
- added J2: DC, Connector_BarrelJack:BarrelJack_GCT_DCJ200-10-A_Horizontal, symbol Connector:Barrel_Jack_Switch
- added J26: ACIAPort, Connector_PinSocket_2.54mm:PinSocket_1x06_P2.54mm_Horizontal, symbol Connector:Conn_01x06_Socket
- added J3: Debug_DATA, Connector_PinHeader_2.54mm:PinHeader_1x08_P2.54mm_Vertical, symbol Connector:Conn_01x08_Socket
- added J4: PWR-SW, Connector_PinHeader_2.54mm:PinHeader_1x03_P2.54mm_Vertical, symbol Connector:Conn_01x03_Socket
- added J5: Debug_ADR0, Connector_PinHeader_2.54mm:PinHeader_1x12_P2.54mm_Vertical, symbol Connector:Conn_01x12_Socket
- added J8: ExpandBus, Connector_PinSocket_2.54mm:PinSocket_2x12_P2.54mm_Horizontal, symbol Connector_Generic:Conn_02x12_Odd_Even
- added J9: ExpandPower, Connector_PinSocket_2.54mm:PinSocket_2x03_P2.54mm_Horizontal, symbol Connector_Generic:Conn_02x03_Odd_Even
- added SW2: SW_Push, Button_Switch_THT:SW_PUSH_6mm_H4.3mm, symbol Switch:SW_Push
- added U1: ATmega328-P, Package_DIP:DIP-28_W7.62mm, symbol MCU_Microchip_ATmega:ATmega328-P
- added U4: 74HC00, Package_DIP:DIP-14_W7.62mm, symbol 74xx:74HC00
- added Y2: Crystal, Crystal:Crystal_HC52-U_Vertical, symbol Device:Crystal
- C1, C10, C11, C12, C13, C15, C16, C17, C2, C24, C25, C26, C3, C4, C5, C6, C7, C8: value 0.1uF -> 0.01uF
- C14: value 0.1uF -> 0.01uF; footprint Capacitor_THT:CP_Radial_D5.0mm_P2.50mm -> Capacitor_THT:C_Disc_D3.4mm_W2.1mm_P2.50mm
- R3, R4, R5, R6: value 10k -> 1K
- SW1: value SW_Push -> RESET
- Y1: footprint crystal:OSC_ECS-2100AX-200 -> Oscillator:Oscillator_DIP-8_LargePads
Connections:
- net CPLD_CLK is gone; now on net CLK: U8.83 (INPUT/GCLK1)
- net NMIB is gone; now on net ROMWEB: U8.30 (IO_22)
- net O0 is gone; now on net D6: U8.46 (IO_34)
- net O1 is gone; now on net D5: U8.48 (IO_35)
- net O10 is gone; now on net A3: U8.58 (IO_44)
- net O11 is gone; now on net A5: U8.60 (IO_45)
- net O12 is gone; now on net A4: U8.61 (IO_46)
- net O13 is gone; now on net A6: U8.63 (IO_47)
- net O15 is gone; now on net A7: U8.65 (IO_49)
- net O2 is gone; now on net D4: U8.49 (IO_36)
- net O3 is gone; now on net D3: U8.50 (IO_37)
- net O4 is gone; now on net D2: U8.51 (IO_38)
- net O5 is gone; now on net D1: U8.52 (IO_39)
- net O6 is gone; now on net A0: U8.54 (IO_40)
- net O7 is gone; now on net D0: U8.55 (IO_41)
- net O8 is gone; now on net A2: U8.56 (IO_42)
- net O9 is gone; now on net A1: U8.57 (IO_43)
- net PORTBD0 is gone; now on net SYS_CONT_D1: U5.10 (PB0)
- net PORTBD1 is gone; now on net SYS_CONT_D2: U5.11 (PB1)
- net PORTBD2 is gone; now on net SYS_CONT_D3: U5.12 (PB2)
- net PORTBD3 is gone; now on net SYS_CONT_D4: U5.13 (PB3)
- net PORTBD4 is gone; now on net SYS_CONT_D5: U5.14 (PB4)
- net PORTBD5 is gone; now on net SYS_CONT_D6: U5.15 (PB5)
- net PORTBD6 is gone; now on net SYS_CONT_D7: U5.16 (PB6)
- net PORTBD7 is gone; now on net SYS_CONT_D8: U5.17 (PB7)
- net A0: now also J5.1 (Pin_1); no longer U8.24 (IO_17)
- net A1: now also J5.2 (Pin_2); no longer U8.25 (IO_18)
- net A10: now also U8.41 (IO_31), J5.11 (Pin_11)
- net A11: now also U8.39 (IO_29), J5.12 (Pin_12)
- net A12: now also U8.31 (IO_23), J13.1 (Pin_1); no longer U8.15 (IO_10)
- net A13: now also U8.35 (IO_26), J13.2 (Pin_2); no longer U8.16 (IO_11)
- net A14: now also U8.34 (IO_25), J13.3 (Pin_3); no longer U8.17 (IO_12)
- net A15: now also U8.33 (IO_24), J13.4 (Pin_4); no longer U8.18 (IO_13)
- net A2: now also J5.3 (Pin_3); no longer U8.27 (IO_19)
- net A3: now also J5.4 (Pin_4); no longer U8.28 (IO_20)
- net A4: now also J5.5 (Pin_5)
- net A5: now also J5.6 (Pin_6)
- net A6: now also J5.7 (Pin_7); no longer U8.20 (IO_14)
- net A7: now also J5.8 (Pin_8); no longer U8.21 (IO_15)
- net A8: now also U8.36 (IO_27), J5.9 (Pin_9); no longer U8.22 (IO_16)
- net A9: now also U8.37 (IO_28), J5.10 (Pin_10)
- net ACIA1CS1: now also U8.18 (IO_13), J12.3 (Pin_3); no longer R4.2
- net ACIA1RX: now also J26.5 (Pin_5)
- net ACIA1TX: now also J26.4 (Pin_4)
- net ACIA2CS1: now also U8.16 (IO_11), J12.1 (Pin_1); no longer R5.2
- net ACIA2RX: now also U1.3 (PD1)
- net ACIA2TX: now also U1.2 (PD0)
- net CA1: now also J7.6 (Pin_6); no longer J7.12 (Pin_12)
- net CA2: now also J7.8 (Pin_8); no longer J7.14 (Pin_14)
- net CB1: now also U8.24 (IO_17); no longer U8.44 (IO_32)
- net CB2: now also U8.22 (IO_16); no longer U8.45 (IO_33)
- net CLK: now also J7.2 (Pin_2), J16.1 (Pin_1), J6.1 (Pin_1), J8.1 (Pin_1); no longer J7.8 (Pin_8), U6.27 (ϕ2), U7.27 (ϕ2), U8.29 (IO_21)
- net D0: now also J3.1 (Pin_1); no longer U8.33 (IO_24)
- net D1: now also J3.2 (Pin_2); no longer U8.34 (IO_25)
- net D2: now also J3.3 (Pin_3); no longer U8.35 (IO_26)
- net D3: now also J3.4 (Pin_4); no longer U8.36 (IO_27)
- net D4: now also J3.5 (Pin_5); no longer U8.37 (IO_28)
- net D5: now also J3.6 (Pin_6); no longer U8.39 (IO_29)
- net D6: now also J3.7 (Pin_7); no longer U8.40 (IO_30)
- net D7: now also U8.45 (IO_33), J3.8 (Pin_8); no longer U8.41 (IO_31)
- net GND: now also C18.2, C25.2, C26.2, J7.18 (Pin_18), R3.2, C19.2, C20.2, C21.2, C22.2, C23.2, C27.2, C28.2, C29.2, C30.2, C31.2, C32.2, C33.2, C34.1, C9.2, J1.10, J10.3 (GND), J10.7 (SHLD_GND), J11.10 (Pin_10), J11.2 (Pin_2), J14.1 (Pin_1), J26.6 (Pin_6), J4.3 (Pin_3), J8.24 (Pin_24), J9.1 (Pin_1), J9.3 (Pin_3), J9.5 (Pin_5), U1.22 (GND), U1.8 (GND), U4.10, U4.12, U4.13, U4.7 (GND), U4.9; no longer C18.1, C25.1, C26.1, J7.4 (Pin_4)
- net IACSB: now also U8.17 (IO_12), J12.2 (Pin_2)
- net IRQ: now also D8.2 (A), D9.2 (A); no longer J7.16 (Pin_16)
- net KEYB_CLK: now also J10.5 (CLK), U4.1, U4.2
- net KEYB_DATA: now also J10.1 (DATA), U1.17 (PB3)
- net RAMCSB: now also U8.44 (IO_32)
- net RAMOEB: now also U8.40 (IO_30)
- net RESB: now also U1.1 (~{RESET}/PC6)
- net ROMCSB: now also U8.29 (IO_21)
- net RWB: now also J7.4 (Pin_4); no longer J7.10 (Pin_10)
- net SYS_CONT_D5: now also R3.1, SW2.1; no longer J7.18 (Pin_18)
- net SYS_CONT_D6: now also J7.12 (Pin_12); no longer J7.17 (Pin_17)
- net SYS_CONT_D7: now also J7.14 (Pin_14)
- net SYS_CONT_D8: now also J7.16 (Pin_16)
- net TCK: now also J11.1 (Pin_1)
- net TDI: now also J11.9 (Pin_9)
- net TDO: now also J11.3 (Pin_3)
- net TMS: now also J11.5 (Pin_5)
- net VCC: now also C18.1, C25.1, C26.1, J7.17 (Pin_17), C20.1, C21.1, C22.1, C23.1, C27.1, C28.1, C29.1, C32.1, C33.1, C34.2, C9.1, D11.2 (A), F1.2, J10.4 (VCC), J15.1 (Pin_1), J17.1 (Pin_1), J18.1 (Pin_1), J19.1 (Pin_1), J20.1 (Pin_1), J21.1 (Pin_1), J22.1 (Pin_1), J23.1 (Pin_1), J24.1 (Pin_1), J26.1 (Pin_1), J8.23 (Pin_23), J9.2 (Pin_2), J9.4 (Pin_4), J9.6 (Pin_6), SW2.2, U1.20 (AVCC), U1.21 (AREF), U1.7 (VCC), U4.14 (VCC); no longer C17.1, C25.2, C26.2, J7.2 (Pin_2), R4.1, R5.1
- net at D2.1 (K): now also U6.26 (~{IRQ})
- net at U7.26 (~{IRQ}): now also D3.1 (K); no longer D5.1 (K)
- net ACIAXT1: now reaches U6.6 (XTAL1), U7.6 (XTAL1), Y3.2
- net ACIAXT1: now also C17.1
- net at D4.1 (K): now also U5.21 (~{IRQ}); no longer U6.26 (~{IRQ})
- net ACIAXT2: now reaches U6.7 (XTAL2), U7.7 (XTAL2), Y3.1
- net ACIAXT2: now also C19.1
- net ACIA2RTS: now reaches U7.8 (~{RTS})
- net ACIA2CTS: now reaches U7.9 (~{CTS})
- net ACIA1RTS: now reaches U6.8 (~{RTS})
- net ACIA1RTS: now also J26.2 (Pin_2)
- net ACIA1CTS: now reaches U6.9 (~{CTS})
- net ACIA1CTS: now also J26.3 (Pin_3)
- net ROMWEB: now reaches U2.27 (~{WE})
- removed net +3V0: J7.6 (Pin_6), R3.2, R6.2
- net IO2 renamed EBB2
- net EBB2: now also J8.16 (Pin_16)
- net IO3 renamed EBB1
- net EBB1: now also J8.18 (Pin_18)
- net IO4 renamed EBA2
- net EBA2: now also J8.15 (Pin_15); no longer R3.1
- net IO5: no longer names the net of R6.1
- net IO5: now also U1.25 (PC2); no longer U8.8 (IO_5)
- net IO6 renamed EBA0
- net EBA0: now also J8.19 (Pin_19)
- net IO7 renamed EBB0
- net EBB0: now also J8.20 (Pin_20)
- net IO8 renamed EBA3
- net EBA3: now also J8.13 (Pin_13)
- net IO9 renamed EBC4
- net EBC4: now also J8.22 (Pin_22)
- net NMIC renamed NMI
- net NMI: now also U8.25 (IO_18)
- net O14 renamed CPRES
- net CPRES: now also J8.2 (Pin_2)
- net O16 renamed EBC2
- net EBC2: now also J8.4 (Pin_4)
- net O17 renamed EBB7
- net EBB7: now also J8.6 (Pin_6)
- net O18 renamed EBC0
- net EBC0: now also J8.3 (Pin_3)
- net O19 renamed EBA7
- net EBA7: now also J8.5 (Pin_5)
- net O20 renamed EBB6
- net EBB6: now also J8.8 (Pin_8)
- net O21 renamed EBA6
- net EBA6: now also J8.7 (Pin_7)
- net O22 renamed EBA5
- net EBA5: now also J8.9 (Pin_9)
- net O23 renamed EBB5
- net EBB5: now also J8.10 (Pin_10)
- net O24 renamed EBB4
- net EBB4: now also J8.12 (Pin_12)
- net O25 renamed EBB3
- net EBB3: now also J8.14 (Pin_14)
- net O26 renamed EBA4
- net EBA4: now also J8.11 (Pin_11)
- net PORTAD0 renamed PORTA0
- net PORTAD1 renamed PORTA1
- net PORTAD2 renamed PORTA2
- net PORTAD3 renamed PORTA3
- net PORTAD4 renamed PORTA4
- net PORTAD5 renamed PORTA5
- net PORTAD6 renamed PORTA6
- net PORTAD7 renamed PORTA7
- net VIA2CS1 renamed VIACS1
- net VIACS1: now also U8.20 (IO_14), J12.4 (Pin_4)
- new net: D11.1 (K), J11.4 (Pin_4)
- new net: R5.1, U1.24 (PC1)
- new net: C31.1, U1.10 (XTAL2/PB7), Y2.1
- new net: U4.3, U4.4, U4.5
- new net: D8.1 (K), U8.21 (IO_15)
- new net: D6.1 (K), F1.1
- new net: D9.1 (K), J8.21 (Pin_21)
- new net: J16.2 (Pin_2), U6.27 (ϕ2)
- new net: U1.19 (PB5), U4.6
- new net: R4.1, U1.23 (PC0)
- new net: C30.1, U1.9 (XTAL1/PB6), Y2.2
- new net: J1.5, J1.6, J1.7, J1.8, J14.2 (Pin_2)
- new net: J2.2, J2.3, J4.2 (Pin_2)
- new net: J6.2 (Pin_2), U7.27 (ϕ2)
- new net: D6.2 (A), J2.1
- new net: D5.1 (K), J7.10 (Pin_10)
- new net EBA1: J8.17 (Pin_17), U8.8 (IO_5)
- new net HSync: J1.13, U1.15 (PB1)
- new net VGA_B: J1.3, R6.2
- new net VGA_G: J1.2, R5.2
- new net VGA_R: J1.1, R4.2
- new net VSync: J1.14, U1.5 (PD3)
- no-connect marks 35 -> 44
Other:
- note added: "Debug"
- note added: "IO Adapters"
- note added: "MAIN"
- note added: "Misc"
- note added: "OK"
- note added: "Power"
- note added: "Terminal"
- note removed: "Step up converters for VIA, ACIA, RAM, ROM"
- title: v6502-Based Homebrew Single Board Computer v2 -> v6502-Based Homebrew Single Board Computer v4
- moved on the sheet: BZ1, D1, D7, J7, R1, R13, R22, R23, R24, R26, U15, U2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
